File: fx2la-mini.kicad_sch (KiCad schematic)
At the start: 45 parts, among them J101 USB_C_Receptacle_USB2.0, J102 Conn_02x11_Counter_Clockwise, U101 CY7C68013A-56LTX, U102 USBLC6-2SC6, U103 MIC5235-3.3YM5-TR, U104 NUF4401MN, U105 NUF4401MN, U106 NUF4401MN, U107 NUF4401MN, Y101 24 MHz

Commit message: Add LED to PA1, update some part numbers that were out of stock now
Parts:
- added D101: LED_Small, LED_SMD:LED_0603_1608Metric, symbol Device:LED_Small
- added R123: 330, passive:R_0402, symbol Device:R_Small
- J102: LCSC (none) -> C725883; MFPN (none) -> X6521WV-2x11H-C30D60
- R102, R103, R104, R105, R106: LCSC C188116 -> C203181; MFPN RM04JTN512 -> CR0402-JW-512GLF
Connections:
- net GND: now also D101.1 (K)
- net LED: now reaches U101.33 (PA0/~{INT0})
- net LED: now also R123.1
- new net: D101.2 (A), R123.2
- no-connect marks 17 -> 16
Changed lines of the file:
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@@
   (no_connect (at 78.74 95.25))
   (no_connect (at 78.74 120.65))
-  (no_connect (at 78.74 110.49))
   (no_connect (at 78.74 125.73))
   (no_connect (at 78.74 118.11))
@@
     (stroke (width 0) (type default))
   )
+  (wire (pts (xy 78.74 110.49) (xy 87.63 110.49))
+    (stroke (width 0) (type default))
+  )
   (wire (pts (xy 269.24 110.49) (xy 266.7 110.49))
     (stroke (width 0) (type default))
@@
     (stroke (width 0) (type default))
   )
+  (wire (pts (xy 92.71 110.49) (xy 96.52 110.49))
+    (stroke (width 0) (type default))
+  )
   (wire (pts (xy 251.46 123.19) (xy 254 123.19))
     (stroke (width 0) (type default))
@@
     (effects (font (size 1.27 1.27)) (justify left bottom))
   )
+  (label "LED" (at 81.28 110.49 0) (fields_autoplaced)
+    (effects (font (size 1.27 1.27)) (justify left bottom))
+  )
   (label "DP_N" (at 64.77 170.18 180) (fields_autoplaced)
     (effects (font (size 1.27 1.27)) (justify right bottom))
@@
     (effects (font (size 1.27 1.27)) (justify left bottom))
   )
+  (symbol (lib_id "Device:LED_Small") (at 99.06 110.49 180) (unit 1)
+    (in_bom yes) (on_board yes) (dnp no) (fields_autoplaced)
+    (property "Reference" "D101" (at 98.9965 106.68 0)
+      (effects (font (size 1.27 1.27)))
+    )
+    (property "Value" "LED_Small" (at 98.9965 106.68 0)
+      (effects (font (size 1.27 1.27)) hide)
+    )
+    (property "Footprint" "LED_SMD:LED_0603_1608Metric" (at 99.06 110.49 90)
+      (effects (font (size 1.27 1.27)) hide)
+    )
+    (property "Datasheet" "~" (at 99.06 110.49 90)
+      (effects (font (size 1.27 1.27)) hide)
+    )
+    (property "MFPN" "NCD0603A1" (at 99.06 110.49 0)
+      (effects (font (size 1.27 1.27)) hide)
+    )
+    (property "Specification" "" (at 99.06 110.49 0)
+      (effects (font (size 1.27 1.27)) hide)
+    )
+    (property "LCSC" "C85323" (at 99.06 110.49 0)
+      (effects (font (size 1.27 1.27)) hide)
+    )
+    (pin "1")
+    (pin "2")
+    (instances
+      (project "fx2la-mini"
+        (path "/102ae594-7aca-4b6c-94aa-7541223a9e55"
+          (reference "D101") (unit 1)
+        )
+      )
+    )
+  )
   (symbol (lib_id "power:+3V3") (at 27.94 109.22 0) (unit 1)
     (in_bom yes) (on_board yes) (dnp no)
@@
       (effects (font (size 1.27 1.27)) hide)
     )
-    (property "MFPN" "RM04JTN512" (at 53.34 163.83 0)
+    (property "MFPN" "CR0402-JW-512GLF" (at 53.34 163.83 0)
       (effects (font (size 1.27 1.27)) hide)
     )
@@
       (effects (font (size 1.27 1.27)) hide)
     )
-    (property "LCSC" "C188116" (at 53.34 163.83 0)
+    (property "LCSC" "C203181" (at 53.34 163.83 0)
       (effects (font (size 1.27 1.27)) hide)
     )
@@
     )
   )
+  (symbol (lib_id "Device:R_Small") (at 90.17 110.49 90) (unit 1)
+    (in_bom yes) (on_board yes) (dnp no) (fields_autoplaced)
+    (property "Reference" "R123" (at 90.17 105.41 90)
+      (effects (font (size 1.27 1.27)))
+    )
+    (property "Value" "330" (at 90.17 107.95 90)
+      (effects (font (size 1.27 1.27)))
+    )
+    (property "Footprint" "passive:R_0402" (at 90.17 110.49 0)
+      (effects (font (size 1.27 1.27)) hide)
+    )
+    (property "Datasheet" "~" (at 90.17 110.49 0)
+      (effects (font (size 1.27 1.27)) hide)
+    )
+    (property "MFPN" "WR04X331JTL" (at 90.17 110.49 0)
+      (effects (font (size 1.27 1.27)) hide)
+    )
+    (property "Specification" "5%" (at 90.17 110.49 0)
+      (effects (font (size 1.27 1.27)) hide)
+    )
+    (property "LCSC" "C168264" (at 90.17 110.49 0)
+      (effects (font (size 1.27 1.27)) hide)
+    )
+    (pin "1")
+    (pin "2")
+    (instances
+      (project "fx2la-mini"
+        (path "/102ae594-7aca-4b6c-94aa-7541223a9e55"
+          (reference "R123") (unit 1)
+        )
+      )
+      (project "crkbd-shockburst"
+        (path "/76f7b6ad-1528-4ee8-9fc0-4578616aebf5/03cbda14-d368-4dde-b0d5-76768308216d"
+          (reference "R206") (unit 1)
+        )
+        (path "/76f7b6ad-1528-4ee8-9fc0-4578616aebf5/3b44a955-2a37-4d30-8a82-5f0155f54e66"
+          (reference "R506") (unit 1)
+        )
+      )
+    )
+  )
   (symbol (lib_id "Connector_Generic:Conn_02x11_Counter_Clockwise") (at 259.08 118.11 0) (unit 1)
     (in_bom yes) (on_board yes) (dnp no) (fields_autoplaced)
@@
       (effects (font (size 1.27 1.27)) hide)
     )
-    (property "MFPN" "" (at 259.08 118.11 0)
+    (property "MFPN" "X6521WV-2x11H-C30D60" (at 259.08 118.11 0)
       (effects (font (size 1.27 1.27)) hide)
     )
@@
       (effects (font (size 1.27 1.27)) hide)
     )
-    (property "LCSC" "" (at 259.08 118.11 0)
+    (property "LCSC" "C725883" (at 259.08 118.11 0)
       (effects (font (size 1.27 1.27)) hide)
     )
@@
       (effects (font (size 1.27 1.27)) hide)
     )
-    (property "MFPN" "RM04JTN512" (at 27.94 111.76 0)
+    (property "MFPN" "CR0402-JW-512GLF" (at 27.94 111.76 0)
       (effects (font (size 1.27 1.27)) hide)
     )
@@
       (effects (font (size 1.27 1.27)) hide)
     )
-    (property "LCSC" "C188116" (at 27.94 111.76 0)
+    (property "LCSC" "C203181" (at 27.94 111.76 0)
       (effects (font (size 1.27 1.27)) hide)
     )
@@
       (effects (font (size 1.27 1.27)) hide)
     )
-    (property "MFPN" "RM04JTN512" (at 31.75 111.76 0)
+    (property "MFPN" "CR0402-JW-512GLF" (at 31.75 111.76 0)
       (effects (font (size 1.27 1.27)) hide)
     )
@@
       (effects (font (size 1.27 1.27)) hide)
     )
-    (property "LCSC" "C188116" (at 31.75 111.76 0)
+    (property "LCSC" "C203181" (at 31.75 111.76 0)
       (effects (font (size 1.27 1.27)) hide)
     )
@@
       (effects (font (size 1.27 1.27)) hide)
     )
-    (property "MFPN" "RM04JTN512" (at 34.29 73.66 0)
+    (property "MFPN" "CR0402-JW-512GLF" (at 34.29 73.66 0)
       (effects (font (size 1.27 1.27)) hide)
     )
@@
       (effects (font (size 1.27 1.27)) hide)
     )
-    (property "LCSC" "C188116" (at 34.29 73.66 0)
+    (property "LCSC" "C203181" (at 34.29 73.66 0)
       (effects (font (size 1.27 1.27)) hide)
     )
@@
     )
   )
+  (symbol (lib_id "power:GND") (at 101.6 110.49 90) (unit 1)
+    (in_bom yes) (on_board yes) (dnp no) (fields_autoplaced)
+    (property "Reference" "#PWR0163" (at 107.95 110.49 0)
+      (effects (font (size 1.27 1.27)) hide)
+    )
+    (property "Value" "GND" (at 105.41 110.4899 90)
+      (effects (font (size 1.27 1.27)) (justify right) hide)
+    )
+    (property "Footprint" "" (at 101.6 110.49 0)
+      (effects (font (size 1.27 1.27)) hide)
+    )
+    (property "Datasheet" "" (at 101.6 110.49 0)
+      (effects (font (size 1.27 1.27)) hide)
+    )
+    (pin "1")
+    (instances
+      (project "fx2la-mini"
+        (path "/102ae594-7aca-4b6c-94aa-7541223a9e55"
+          (reference "#PWR0163") (unit 1)
+        )
+      )
+    )
+  )
   (symbol (lib_id "Device:R_Small") (at 53.34 161.29 270) (unit 1)
     (in_bom yes) (on_board yes) (dnp no) (fields_autoplaced)
@@
       (effects (font (size 1.27 1.27)) hide)
     )
-    (property "MFPN" "RM04JTN512" (at 53.34 161.29 0)
+    (property "MFPN" "CR0402-JW-512GLF" (at 53.34 161.29 0)
       (effects (font (size 1.27 1.27)) hide)
     )
@@
       (effects (font (size 1.27 1.27)) hide)
     )
-    (property "LCSC" "C188116" (at 53.34 161.29 0)
+    (property "LCSC" "C203181" (at 53.34 161.29 0)
       (effects (font (size 1.27 1.27)) hide)
     )
